Commit message: fix(linker-l20): align AnyDex mapping and MCP axes

File: assets/dex_hand/linker_l20/left_hand.urdf.xacro (robot description, xacro)
@@ -560,5 +560,5 @@
       <parent link="left_hand_base_link" />
       <child link="left_if_mcp_roll_link" />
-      <axis xyz="-1 0 0" />
+      <axis xyz="1 0 0" />
       <limit lower="-0.23" upper="0.23" effort="100" velocity="1" />
     </joint>
@@ -589,5 +589,5 @@
       <parent link="left_hand_base_link" />
       <child link="left_mf_mcp_roll_link" />
-      <axis xyz="-1 0 0" />
+      <axis xyz="1 0 0" />
       <limit lower="-0.23" upper="0.23" effort="100" velocity="1" />
     </joint>
@@ -618,5 +618,5 @@
       <parent link="left_hand_base_link" />
       <child link="left_rf_mcp_roll_link" />
-      <axis xyz="-1 0 0" />
+      <axis xyz="1 0 0" />
       <limit lower="-0.23" upper="0.23" effort="100" velocity="1" />
     </joint>
@@ -647,5 +647,5 @@
       <parent link="left_hand_base_link" />
       <child link="left_lf_mcp_roll_link" />
-      <axis xyz="-1 0 0" />
+      <axis xyz="1 0 0" />
       <limit lower="-0.23" upper="0.23" effort="100" velocity="1" />
     </joint>

File: assets/dex_hand/linker_l20/linker_l20_left_vis.urdf (robot description, URDF)
Before this commit: robot linker_l20_left, 29 links, 28 joints
Joints:
- joint LEFT_IF_MCP_ROLL: axis -1 0 0 -> 1 0 0
- joint LEFT_LF_MCP_ROLL: axis -1 0 0 -> 1 0 0
- joint LEFT_MF_MCP_ROLL: axis -1 0 0 -> 1 0 0
- joint LEFT_RF_MCP_ROLL: axis -1 0 0 -> 1 0 0

File: assets/dex_hand/linker_l20/linker_l20_right_vis.urdf (robot description, URDF)
Before this commit: robot linker_l20_right, 29 links, 28 joints
Joints:
- joint RIGHT_IF_MCP_ROLL: axis 1 0 0 -> -1 0 0
- joint RIGHT_LF_MCP_ROLL: axis 1 0 0 -> -1 0 0
- joint RIGHT_MF_MCP_ROLL: axis 1 0 0 -> -1 0 0
- joint RIGHT_RF_MCP_ROLL: axis 1 0 0 -> -1 0 0

File: assets/dex_hand/linker_l20/right_hand.urdf.xacro (robot description, xacro)
@@ -560,5 +560,5 @@
       <parent link="right_hand_base_link" />
       <child link="right_if_mcp_roll_link" />
-      <axis xyz="1 0 0" />
+      <axis xyz="-1 0 0" />
       <limit lower="-0.23" upper="0.23" effort="1" velocity="100" />
     </joint>
@@ -589,5 +589,5 @@
       <parent link="right_hand_base_link" />
       <child link="right_mf_mcp_roll_link" />
-      <axis xyz="1 0 0" />
+      <axis xyz="-1 0 0" />
       <limit lower="-0.23" upper="0.23" effort="1" velocity="100" />
     </joint>
@@ -618,5 +618,5 @@
       <parent link="right_hand_base_link" />
       <child link="right_rf_mcp_roll_link" />
-      <axis xyz="1 0 0" />
+      <axis xyz="-1 0 0" />
       <limit lower="-0.23" upper="0.23" effort="1" velocity="100" />
     </joint>
@@ -647,5 +647,5 @@
       <parent link="right_hand_base_link" />
       <child link="right_lf_mcp_roll_link" />
-      <axis xyz="1 0 0" />
+      <axis xyz="-1 0 0" />
       <limit lower="-0.23" upper="0.23" effort="1" velocity="100" />
     </joint>
